File: Hardware/MyoWare_LED_Shield.sch (EAGLE design)
At the start: 25 parts, among them U1 MCP73831, U2 LM3914V

Commit message: Improved micro-B DFM & fixed alignment silk
Connections:
- new net D+: JP4.D+
- new net D-: JP4.D-
- new net ID: JP4.ID
- new net SHIELD: JP4.SHIELD
Changed lines of the file:
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@@
 </plain>
 <instances>
-<instance part="JP2" gate="G$1" x="33.02" y="147.32" rot="MR180"/>
+<instance part="JP2" gate="J$1" x="33.02" y="147.32" rot="MR180"/>
 <instance part="D3" gate="G$1" x="160.02" y="63.5" smashed="yes">
 <attribute name="NAME" x="154.94" y="76.2" size="0.8128" layer="95"/>
@@
 </instance>
 <instance part="GND1" gate="1" x="111.76" y="33.02"/>
-<instance part="JP1" gate="G$1" x="33.02" y="127" rot="MR180"/>
+<instance part="JP1" gate="J$1" x="33.02" y="127" rot="MR180"/>
 <instance part="MODE" gate="G$1" x="91.44" y="76.2" smashed="yes" rot="R90">
 <attribute name="NAME" x="89.662" y="72.898" size="1.778" layer="95" rot="R90"/>
@@
 </segment>
 <segment>
-<pinref part="JP1" gate="G$1" pin="3"/>
+<pinref part="JP1" gate="J$1" pin="3"/>
 <wire x1="40.64" y1="124.46" x2="43.18" y2="124.46" width="0.1524" layer="91"/>
 <pinref part="GND2" gate="1" pin="GND"/>
@@
 <pinref part="GND10" gate="1" pin="GND"/>
 <wire x1="50.8" y1="144.78" x2="50.8" y2="147.32" width="0.1524" layer="91"/>
-<pinref part="JP2" gate="G$1" pin="2"/>
+<pinref part="JP2" gate="J$1" pin="2"/>
 <wire x1="50.8" y1="147.32" x2="40.64" y2="147.32" width="0.1524" layer="91"/>
 </segment>
@@
 <segment>
 <wire x1="40.64" y1="144.78" x2="43.18" y2="144.78" width="0.1524" layer="91"/>
-<pinref part="JP2" gate="G$1" pin="3"/>
+<pinref part="JP2" gate="J$1" pin="3"/>
 <label x="43.18" y="144.78" size="1.27" layer="95" xref="yes"/>
 </segment>
@@
 <pinref part="+VS1" gate="G$1" pin="1.0V"/>
 <wire x1="43.18" y1="152.4" x2="43.18" y2="149.86" width="0.1524" layer="91"/>
-<pinref part="JP2" gate="G$1" pin="1"/>
+<pinref part="JP2" gate="J$1" pin="1"/>
 <wire x1="40.64" y1="149.86" x2="43.18" y2="149.86" width="0.1524" layer="91"/>
 </segment>
@@
 <segment>
 <wire x1="43.18" y1="127" x2="40.64" y2="127" width="0.1524" layer="91"/>
-<pinref part="JP1" gate="G$1" pin="2"/>
+<pinref part="JP1" gate="J$1" pin="2"/>
 <label x="43.18" y="127" size="1.27" layer="95" xref="yes"/>
 </segment>
@@
 <segment>
 <wire x1="43.18" y1="129.54" x2="40.64" y2="129.54" width="0.1524" layer="91"/>
-<pinref part="JP1" gate="G$1" pin="1"/>
+<pinref part="JP1" gate="J$1" pin="1"/>
 <label x="43.18" y="129.54" size="1.27" layer="95" xref="yes"/>
 </segment>
@@
 </segment>
 </net>
+<net name="SHIELD" class="0">
+<segment>
+<pinref part="JP4" gate="G$1" pin="SHIELD"/>
+<wire x1="88.9" y1="154.94" x2="86.36" y2="154.94" width="0.1524" layer="91"/>
+<label x="86.36" y="154.94" size="1.27" layer="91" rot="R180" xref="yes"/>
+</segment>
+</net>
+<net name="D-" class="0">
+<segment>
+<pinref part="JP4" gate="G$1" pin="D-"/>
+<wire x1="104.14" y1="157.48" x2="106.68" y2="157.48" width="0.1524" layer="91"/>
+<label x="106.68" y="157.48" size="1.27" layer="91" xref="yes"/>
+</segment>
+</net>
+<net name="D+" class="0">
+<segment>
+<pinref part="JP4" gate="G$1" pin="D+"/>
+<wire x1="104.14" y1="154.94" x2="106.68" y2="154.94" width="0.1524" layer="91"/>
+<label x="106.68" y="154.94" size="1.27" layer="91" xref="yes"/>
+</segment>
+</net>
+<net name="ID" class="0">
+<segment>
+<pinref part="JP4" gate="G$1" pin="ID"/>
+<wire x1="104.14" y1="152.4" x2="106.68" y2="152.4" width="0.1524" layer="91"/>
+<label x="106.68" y="152.4" size="1.27" layer="91" xref="yes"/>
+</segment>
+</net>
