File: Hardware/MyoWare_LED_Shield.sch (EAGLE design)
At the start: 25 parts, among them U1 MCP73831, U2 LM3914V

Commit message: Change charge done LED to green
Parts:
- D2: value RED -> GREEN; device SparkFun-LED:LED-RED0603 -> SparkFun-LED:LED-GREEN0603
Changed lines of the file:
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@@
 <part name="GND6" library="SparkFun" deviceset="GND" device=""/>
 <part name="GND7" library="SparkFun" deviceset="GND" device=""/>
-<part name="D2" library="SparkFun-LED" deviceset="LED-RED" device="0603" value="RED"/>
+<part name="D2" library="SparkFun-LED" deviceset="LED-GREEN" device="0603" value="GREEN"/>
 <part name="R5" library="SparkFun-Resistors" deviceset="330OHM1/10W1%(0603)" device="" value="330"/>
 <part name="GND8" library="SparkFun" deviceset="GND" device=""/>
