File: Hardware/MyoWare_LED_Shield.brd (EAGLE design)
At the start: 52.3 x 21.8 mm, 27 parts, among them U1 MCP73831, U2 LM3914V

Commit message: Change charge done LED to green
Parts:
- D2: value RED -> GREEN
Changed lines of the file:
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@@
 </element>
 <element name="JP3" library="SparkFun-Connectors" package="1X02_NO_SILK" value="LiPo" x="49.4665" y="5.0165" rot="R225"/>
-<element name="D2" library="SparkFun-LED" package="LED-0603" value="RED" x="48.5775" y="15.9385" rot="MR90">
-<attribute name="PROD_ID" value="DIO-00819" x="48.5775" y="15.9385" size="1.778" layer="28" rot="MR90" display="off"/>
+<element name="D2" library="SparkFun-LED" package="LED-0603" value="GREEN" x="48.5775" y="15.9385" rot="MR90">
+<attribute name="PROD_ID" value="DIO-00821" x="48.5775" y="15.9385" size="1.778" layer="28" rot="MR90" display="off"/>
 </element>
 <element name="R5" library="SparkFun-Resistors" package="0603-RES" value="330" x="43.561" y="14.351" rot="MR180">
